File: 1. Hardware/RaZbyBoard-DomoCAN-Bridge-v1.0.kicad_pcb (KiCad board)
At the start: 2 copper layers, 23 parts, among them IC1 MCP2515, IC2 MCP2551, IC3 DS1307, P1 Raspberry Pi, P2 Power, P3 CAN, P4 1 Wire, P5 RTC Bat., P999 CONN_1, X1 16MHz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

Commit message: v1
Parts:
- added P6: CONN_4, PIN_ARRAY_4x1, F.Cu at (142.1, 112.2)
Routing:
- net GND: track 439.4 -> 485.1 mm
- net 5.0 V: track 117.4 -> 150.6 mm
- net I2C_SDA: track 52.1 -> 53.3 mm
